File: pcb/a3000_rom_emulator.kicad_pcb (KiCad board)
At the start: 4 copper layers, 43.2 x 78.7 mm, 112 parts, among them T1 rom_5V

Commit message: PCB updates I did a while ago -- I'm not even sure what's in here...
Other:
- board text added: "JLCJLCJLCJLC"
