File: pcb/a3000_rom_emulator.kicad_pcb (KiCad board)
At the start: 4 copper layers, 43.2 x 78.7 mm, 112 parts, among them T1 rom_5V

Commit message: pcb: Update to KiCad 9, fix Makefile to build fab outputs again
Other:
- net class Default removed
- net class Flash Control removed
- net class Power removed
- board text added: "JLCJLCJLCJLC"
