File: riscpc_adapter_pcb/riscpc_adapter.kicad_pcb (KiCad board)
At the start: 2 copper layers, 58.4 x 101.6 mm, 108 parts

Commit message: PCB updates I did a while ago -- I'm not even sure what's in here...
Parts:
- moved RPCROM1 1.27 mm to (130.0, 137.2)
- moved staple_single83 0.74 mm to (135.6, 111.9)
Routing:
- net D2: track 107.6 -> 108.9 mm
- net D3: track 131.8 -> 133.1 mm
- net D8: track 78.7 -> 80.0 mm
- net D11: track 113.7 -> 115.0 mm
- net D0: track 94.8 -> 96.1 mm
- net D9: track 89.6 -> 90.9 mm
- net D7: track 94.2 -> 95.5 mm
- net D5: track 111.8 -> 113.0 mm
- net D4: track 120.9 -> 122.2 mm
- net D15: track 69.1 -> 70.4 mm
- net D14: track 86.9 -> 88.2 mm
- net D13: track 95.8 -> 97.0 mm
- net D10: track 93.1 -> 94.3 mm
- net A15: track 53.3 -> 54.6 mm
- net A13: track 76.2 -> 77.4 mm
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Other:
- board size 58.4 x 101.6 mm -> 59.7 x 101.6 mm
